File: reload.brd (EAGLE design)
At the start: 49.2 x 30.5 mm, 22 parts, among them IC1 MCP6002, IC2 LP2950Z, Q1 BTS117

Commit message: Started modding. Still need to add chips.
Parts:
- removed IC1: MCP6002, SparkFun-AnalogIC:DIP08
- removed IC2: LP2950Z, linear:TO92
- removed R2: 1k, nickparts:TRIMPOT-3MM-2
- removed R4, R5: 10k 1%, SparkFun-Passives:AXIAL-0.3
- removed TP1, TP2: (no value), microbuilder:1X01_ROUND
- added U1: MCP1790-3302E/DB, Microchip_By_element14_Batch_1:SOT230P700X180-4N
- added U2: MCP6V01-E/SN, Microchip_By_element14_Batch_1:SOIC127P600X175-8N
- C2: value 10u -> 1u
- R3: value 162k -> 180k 0.1%
Connections:
- removed net IREF: IC1.7, R4.P$1, TP1.1
- removed net N$1: IC1.1, R7.P$2
- removed net N$4: IC1.3, R6.P$2
- removed net N$5: IC1.6, R2.2
- removed net N$6: R2.1, R5.P$1
- removed net N$7: R2.3, R4.P$2
- removed net SENSE: IC1.2, IC1.5, Q1.3, R1.P$2
- new net N$3: C1.1, U2.7
- new net VINA+: R6.P$2, U2.3
- new net VINA-: Q1.3, R1.P$2, U2.2
- new net VOUTA: R7.P$2, U2.6
- net GND: now also U1.2, U1.4, U2.4; no longer IC1.4, IC2.2, R5.P$2, TP2.1
- net N$8: now also U1.1; no longer IC2.3
- net VCC: no longer C1.1, IC1.8, IC2.1
Routing:
- net SENSE: track 58.0 -> 0.00 mm
- net VCC: track 55.8 -> 30.4 mm
- net GND: track 91.1 -> 68.8 mm
- net N$4: track 16.5 -> 0.00 mm
- net VINA+: track 0.00 -> 14.3 mm
- net N$1: track 14.1 -> 0.00 mm
- net VOUTA: track 0.00 -> 12.3 mm
- net IREF: track 9.04 -> 0.00 mm
- net N$7: track 7.65 -> 0.00 mm
- net N$5: track 4.66 -> 0.00 mm
- net N$6: track 2.91 -> 0.00 mm
- net N$8: track 15.5 -> 13.3 mm
