File: reload.sch (EAGLE design)
At the start: 20 parts, among them IC1 MCP6002, IC2 LP2950Z, Q1 BTS117

Commit message: Started modding. Still need to add chips.
Parts:
- removed IC1: MCP6002, SparkFun-AnalogIC:LM358
- removed IC2: LP2950Z, linear:LP2950Z
- removed R2: 1k, nickparts:TRIMPOT3MM-2
- removed R4, R5: 10k 1%, SparkFun-Passives:RESISTORAXIAL-0.3
- removed TP1, TP2: (no value), microbuilder:TESTPOINT0.1"
- added U1: MCP1790-3302E/DB, Microchip_By_element14_Batch_1:MCP1790-3302E/DB
- added U2: MCP6V01-E/SN, Microchip_By_element14_Batch_1:MCP6V01-E/SN
- C2: value 10u -> 1u
- R3: value 162k -> 180k 0.1%
Connections:
- removed net IREF: IC1G$2.OUT, R4.1, TP1.P$1
- removed net N$1: IC1G$1.OUT, R7.2
- removed net N$4: IC1G$1.+IN, R6.S
- removed net N$5: IC1G$2.-IN, R2.WIPER
- removed net N$6: R2.CCW, R5.1
- removed net N$7: R2.CW, R4.2
- removed net SENSE: IC1G$1.-IN, IC1G$2.+IN, Q1.S, R1.2
- new net N$3: C1.1, U2.VDD
- new net VINA+: R6.S, U2.VIN+
- new net VINA-: Q1.S, R1.2, U2.VIN-
- new net VOUTA: R7.2, U2.VOUT
- net GND: now also U1.GND_(TAB), U1.GND_(TAB)_2, U2.VSS; no longer IC1G$1.V-, IC2.GND, R5.2, TP2.P$1
- net N$8: now also U1.VIN; no longer IC2.I
- net VCC: no longer C1.1, IC1G$1.V+, IC2.O
Other:
- moved on the sheet: C1, C2, C3, D1, R3
